Commit message: update wamv urdf

File: wamv_gazebo/urdf/components/ball_shooter.xacro (robot description, xacro)
@@ -45,5 +45,5 @@
       </inertial>
     </link>
-    <joint name="${namespace}/${name}_base_joint" type="revolute">
+    <joint name="${namespace}/${name}_base_joint" type="fixed">
       <axis xyz="0 0 1"/>
       <limit effort="1000.0" lower="0.0" upper="0" velocity="0"/>
@@ -52,5 +52,5 @@
       <child link="${namespace}/${name}_base_link"/>
     </joint>
-    <joint name="${namespace}/${name}_launcher_joint" type="revolute">
+    <joint name="${namespace}/${name}_launcher_joint" type="fixed">
       <axis xyz="0 0 1"/>
       <limit effort="1000.0" lower="0.0" upper="0" velocity="0"/>

File: wamv_gazebo/urdf/components/wamv_gps.xacro (robot description, xacro)
@@ -27,5 +27,5 @@
       </inertial>
     </link>
-    <joint name="${namespace}/${name}_joint" type="revolute">
+    <joint name="${namespace}/${name}_joint" type="fixed">
       <axis xyz="0 0 1"/>
       <limit effort="1000.0" lower="0.0" upper="0" velocity="0"/>

File: wamv_gazebo/urdf/components/wamv_imu.xacro (robot description, xacro)
@@ -16,5 +16,5 @@
       </inertial>
     </link>
-    <joint name="${namespace}/${name}_joint" type="revolute">
+    <joint name="${namespace}/${name}_joint" type="fixed">
       <axis xyz="0 0 1"/>
       <limit effort="1000.0" lower="0.0" upper="0" velocity="0"/>
