Commit message: update on vrx

File: wamv_gazebo/urdf/wamv_gazebo.urdf.xacro (robot description, xacro)
@@ -80,5 +80,5 @@
       <joint name="wamv_external_riser" type="prismatic">
         <parent>world</parent>
-        <child>wamv_external_link</child>
+        <child>wamv/base_link</child>
         <axis>
           <limit>
@@ -136,6 +136,7 @@
       <xacro:cpu_cases position="-0.15 0 1.53" orientation="0 0 0"/>
       <!-- Add a stereo camera pair -->
-      <xacro:wamv_camera name="front_left_camera" y="0.1" x="0.75" P="${radians(15)}" />
-      <xacro:wamv_camera name="front_right_camera" y="-0.1" x="0.75" P="${radians(15)}" />
+      <!-- <xacro:wamv_camera name="front_left_camera" y="0.1" x="0.75" P="${radians(15)}" />
+      <xacro:wamv_camera name="front_right_camera" y="-0.1" x="0.75" P="${radians(15)}" /> -->
+      <xacro:wamv_camera name="front_middle_camera" y="0.0" x="0.75" P="${radians(15)}" />
       <!-- Add a camera facing right -->
       <xacro:wamv_camera name="middle_right_camera" y="-0.45" P="${radians(15)}" Y="${radians(-90)}" post_Y="${radians(-90)}" />
