Commit message: on vrx

File: wamv_description/urdf/wamv_base.urdf.xacro (robot description, xacro)
@@ -5,5 +5,5 @@
   <xacro:property name="namespace" value="$(arg namespace)" scope="global" />
   <!-- Macro for creating the main collisions as simple shapes. -->
-  <xacro:macro name="main_collisions" params="prefix reflect:=1">
+  <xacro:macro name="main_collisions" params="prefix reflect:=10">
     <!-- Main float -->
     <collision name="${prefix}_float">

File: wave_gazebo/world_models/ocean_waves/model.xacro (robot description, xacro)
@@ -17,5 +17,5 @@
 -->
 <world xmlns:xacro="http://ros.org/wiki/xacro">
-  <xacro:macro name="ocean_waves" params="gain:=0.1 period:=5
+  <xacro:macro name="ocean_waves" params="gain:=0.7 period:=5
                      direction_x:=1.0 direction_y:=0.0
                      angle:=0.4 scale:=1.5">
