Commit message: update master thesis world on vrx

File: vrx_gazebo/worlds/master_thesis.world.xacro (robot description, xacro)
@@ -31,95 +31,15 @@
     <include>
       <uri>model://robotx_light_buoy</uri>
-      <pose>-511 218 0.25 0 0 3.14</pose>
+      <pose>-500 224 0.25 0 0 3.14</pose>
     </include>
     <!-- The 2022 dock with the placards -->
     <include>
       <uri>model://dock_2022</uri>
-      <pose>-554 233 0 0 0 3.14</pose>
+      <pose>-550 233 0 0 0 3.14</pose>
     </include>
-    <!-- Plugin to detect if the projectile entered the hole -->
-    <!-- Debug: Run this command to face this hole -->
-    <!-- gz model -m wamv -x -555.21 -y 229.75 -z 0 -Y 3.14159 -->
-    <plugin name="contain_placard1_big_plugin" filename="libContainPlugin.so">
-      <enabled>true</enabled>
-      <entity>blue_projectile::link</entity>
-      <namespace>vrx/dock_2022_placard1_big_hole</namespace>
-      <pose frame="robotx_dock_2022::dock_2022_placard1::link_symbols">0.6 -0.27 1.33 0 0 0</pose>
-      <geometry>
-        <box>
-          <size>0.5 0.5 0.5</size>
-        </box>
-      </geometry>
-    </plugin>
-    <!-- Plugin to detect if the projectile entered the hole -->
-    <!-- Debug: Run this command to face this hole -->
-    <!-- gz model -m wamv -x -555.28 -y 230.32 -z 0 -Y 3.01159 -->
-    <plugin name="contain_placard1_small_plugin" filename="libContainPlugin.so">
-      <enabled>true</enabled>
-      <entity>blue_projectile::link</entity>
-      <namespace>vrx/dock_2022_placard1_small_hole</namespace>
-      <pose frame="robotx_dock_2022::dock_2022_placard1::link_symbols">-0.6 -0.27 1.33 0 0 0</pose>
-      <geometry>
-        <box>
-          <size>0.25 0.5 0.25</size>
-        </box>
-      </geometry>
-    </plugin>
-    <!-- Plugin to detect if the projectile entered the hole -->
-    <!-- Debug: Run this command to face this hole -->
-    <!-- gz model -m wamv -x -555.21 -y 223.75 -z 0 -Y 3.14159 -->
-    <plugin name="contain_placard2_big_plugin" filename="libContainPlugin.so">
-      <enabled>true</enabled>
-      <entity>blue_projectile::link</entity>
-      <namespace>vrx/dock_2022_placard2_big_hole</namespace>
-      <pose frame="robotx_dock_2022::dock_2022_placard2::link_symbols">0.6 -0.27 1.33 0 0 0</pose>
-      <geometry>
-        <box>
-          <size>0.5 0.5 0.5</size>
-        </box>
-      </geometry>
-    </plugin>
-    <!-- Plugin to detect if the projectile entered the hole -->
-    <!-- Debug: Run this command to face this hole -->
-    <!-- gz model -m wamv -x -555.25 -y 223.75 -z 0 -Y 2.91159 -->
-    <plugin name="contain_placard2_small_plugin" filename="libContainPlugin.so">
-      <enabled>true</enabled>
-      <entity>blue_projectile::link</entity>
-      <namespace>vrx/dock_2022_placard2_small_hole</namespace>
-      <pose frame="robotx_dock_2022::dock_2022_placard2::link_symbols">-0.6 -0.27 1.33 0 0 0</pose>
-      <geometry>
-        <box>
-          <size>0.25 0.5 0.25</size>
-        </box>
-      </geometry>
-    </plugin>
-    <!-- Plugin to detect if the projectile entered the hole -->
-    <!-- Debug: Run this command to face this hole -->
-    <!-- gz model -m wamv -x -555.25 -y 217.75 -z 0 -Y 3.14159 -->
-    <plugin name="contain_placard3_big_plugin" filename="libContainPlugin.so">
-      <enabled>true</enabled>
-      <entity>blue_projectile::link</entity>
-      <namespace>vrx/dock_2022_placard3_big_hole</namespace>
-      <pose frame="robotx_dock_2022::dock_2022_placard3::link_symbols">0.6 -0.27 1.33 0 0 0</pose>
-      <geometry>
-        <box>
-          <size>0.5 0.5 0.5</size>
-        </box>
-      </geometry>
-    </plugin>
-    <!-- Plugin to detect if the projectile entered the hole -->
-    <!-- Debug: Run this command to face this hole -->
-    <!-- gz model -m wamv -x -555.25 -y 217.75 -z 0 -Y 2.89159 -->
-    <plugin name="contain_placard3_small_plugin" filename="libContainPlugin.so">
-      <enabled>true</enabled>
-      <entity>blue_projectile::link</entity>
-      <namespace>vrx/dock_2022_placard3_small_hole</namespace>
-      <pose frame="robotx_dock_2022::dock_2022_placard3::link_symbols">-0.6 -0.27 1.33 0 0 0</pose>
-      <geometry>
-        <box>
-          <size>0.25 0.5 0.25</size>
-        </box>
-      </geometry>
-    </plugin>
+    <include>
+      <uri>model://dock_2022_base</uri>
+      <pose>-450 215 0 0 0 0</pose>
+    </include>
     <!-- The scoring plugin -->
     <plugin name="scan_dock_deliver_scoring_plugin"
@@ -154,5 +74,5 @@
           <external_activation_topic>/vrx/dock_2022/bay_1_external/contain</external_activation_topic>
           <symbol_topic>/vrx/dock_2022_placard1/symbol</symbol_topic>
-          <min_dock_time>10.0</min_dock_time>
+          <min_dock_time>5.0</min_dock_time>
           <dock_allowed>${bay1_allowed}</dock_allowed>
           <symbol>${bay1_symbol}</symbol>
@@ -163,5 +83,5 @@
           <external_activation_topic>/vrx/dock_2022/bay_2_external/contain</external_activation_topic>
           <symbol_topic>/vrx/dock_2022_placard2/symbol</symbol_topic>
-          <min_dock_time>10.0</min_dock_time>
+          <min_dock_time>5.0</min_dock_time>
           <dock_allowed>${bay2_allowed}</dock_allowed>
           <symbol>${bay2_symbol}</symbol>
@@ -172,5 +92,5 @@
           <external_activation_topic>/vrx/dock_2022/bay_3_external/contain</external_activation_topic>
           <symbol_topic>/vrx/dock_2022_placard3/symbol</symbol_topic>
-          <min_dock_time>10.0</min_dock_time>
+          <min_dock_time>5.0</min_dock_time>
           <dock_allowed>${bay3_allowed}</dock_allowed>
           <symbol>${bay3_symbol}</symbol>
@@ -261,5 +181,5 @@
       </geometry>
     </plugin>
-    <plugin filename="libContainPlugin.so" name="vehicle_docked_bay3_exterior">
+    <plugin name="vehicle_docked_bay3_exterior" filename="libContainPlugin.so">
       <entity>wamv::wamv/base_link</entity>
       <namespace>vrx/dock_2022/bay_3_external</namespace>

Commit message: update vrx on vrx

File: vrx_gazebo/worlds/master_thesis.world.xacro (robot description, xacro)
@@ -29,166 +29,24 @@
     </xacro:usv_wind_gazebo>
     <!-- The light buoy -->
-    <include>
+    <!-- <include>
       <uri>model://robotx_light_buoy</uri>
       <pose>-500 224 0.25 0 0 3.14</pose>
-    </include>
+    </include> -->
     <!-- The 2022 dock with the placards -->
+    <!-- <include>
+      <name>dock_1</name>
+      <uri>model://dock_2022</uri>
+      <pose>-550 233 0 0 0 3.14</pose>
+    </include> -->
     <include>
-      <uri>model://dock_2022</uri>
+      <name>dock_1</name>
+      <uri>model://dock_2022_base</uri>
       <pose>-550 233 0 0 0 3.14</pose>
     </include>
     <include>
+      <name>dock_2</name>
       <uri>model://dock_2022_base</uri>
       <pose>-450 215 0 0 0 0</pose>
     </include>
-    <!-- The scoring plugin -->
-    <plugin name="scan_dock_deliver_scoring_plugin"
-            filename="libscan_dock_scoring_plugin.so">
-      <!-- Parameters for scoring_plugin -->
-      <vehicle>wamv</vehicle>
-      <task_name>scan_dock_deliver</task_name>
-      <initial_state_duration>3</initial_state_duration>
-      <ready_state_duration>3</ready_state_duration>
-      <running_state_duration>300</running_state_duration>
-      <release_joints>
-        <joint>
-          <name>wamv_external_pivot_joint</name>
-        </joint>
-        <joint>
-          <name>wamv_external_riser</name>
-        </joint>
-      </release_joints>
-      <!-- Color sequence checker -->
-      <robot_namespace>vrx</robot_namespace>
-      <color_sequence_service>scan_dock_deliver/color_sequence</color_sequence_service>
-      <color_1>${color_1}</color_1>
-      <color_2>${color_2}</color_2>
-      <color_3>${color_3}</color_3>
-      <!-- Dock checkers -->
-      <dock_bonus_points>15</dock_bonus_points>
-      <correct_dock_bonus_points>5</correct_dock_bonus_points>
-      <bays>
-        <bay>
-          <name>bay1</name>
-          <internal_activation_topic>/vrx/dock_2022/bay_1/contain</internal_activation_topic>
-          <external_activation_topic>/vrx/dock_2022/bay_1_external/contain</external_activation_topic>
-          <symbol_topic>/vrx/dock_2022_placard1/symbol</symbol_topic>
-          <min_dock_time>5.0</min_dock_time>
-          <dock_allowed>${bay1_allowed}</dock_allowed>
-          <symbol>${bay1_symbol}</symbol>
-        </bay>
-        <bay>
-          <name>bay2</name>
-          <internal_activation_topic>/vrx/dock_2022/bay_2/contain</internal_activation_topic>
-          <external_activation_topic>/vrx/dock_2022/bay_2_external/contain</external_activation_topic>
-          <symbol_topic>/vrx/dock_2022_placard2/symbol</symbol_topic>
-          <min_dock_time>5.0</min_dock_time>
-          <dock_allowed>${bay2_allowed}</dock_allowed>
-          <symbol>${bay2_symbol}</symbol>
-        </bay>
-        <bay>
-          <name>bay3</name>
-          <internal_activation_topic>/vrx/dock_2022/bay_3/contain</internal_activation_topic>
-          <external_activation_topic>/vrx/dock_2022/bay_3_external/contain</external_activation_topic>
-          <symbol_topic>/vrx/dock_2022_placard3/symbol</symbol_topic>
-          <min_dock_time>5.0</min_dock_time>
-          <dock_allowed>${bay3_allowed}</dock_allowed>
-          <symbol>${bay3_symbol}</symbol>
-        </bay>
-      </bays>
-      <!-- Shooting targets -->
-      <targets>
-        <!-- Placard #1 -->
-        <target>
-          <topic>vrx/dock_2022_placard1_big_hole/contain</topic>
-          <bonus_points>5</bonus_points>
-        </target>
-        <target>
-          <topic>vrx/dock_2022_placard1_small_hole/contain</topic>
-          <bonus_points>10</bonus_points>
-        </target>
-        <!-- Placard #2 -->
-        <target>
-          <topic>vrx/dock_2022_placard2_big_hole/contain</topic>
-          <bonus_points>5</bonus_points>
-        </target>
-        <target>
-          <topic>vrx/dock_2022_placard2_small_hole/contain</topic>
-          <bonus_points>10</bonus_points>
-        </target>
-        <!-- Placard #3 -->
-        <target>
-          <topic>vrx/dock_2022_placard3_big_hole/contain</topic>
-          <bonus_points>5</bonus_points>
-        </target>
-        <target>
-          <topic>vrx/dock_2022_placard3_small_hole/contain</topic>
-          <bonus_points>10</bonus_points>
-        </target>
-      </targets>
-    </plugin>
-    <!-- Triggers a message when the vehicle enters and exits the bay #1 -->
-    <plugin name="vehicle_docked_bay1" filename="libContainPlugin.so">
-      <entity>wamv::wamv/base_link</entity>
-      <namespace>vrx/dock_2022/bay_1</namespace>
-      <pose frame="robotx_dock_2022::dock_2022_placard1::placard::link">0 -4.5 -1.5 0 0 0</pose>
-      <geometry>
-        <box>
-          <size>1.5 4 2</size>
-        </box>
-      </geometry>
-    </plugin>
-    <plugin name="vehicle_docked_bay1_exterior" filename="libContainPlugin.so">
-      <entity>wamv::wamv/base_link</entity>
-      <namespace>vrx/dock_2022/bay_1_external</namespace>
-      <pose frame="robotx_dock_2022::dock_2022_placard1::placard::link">0 -9.5 -1.5 0 0 0</pose>
-      <geometry>
-        <box>
-          <size>5.5 1.5 2</size>
-        </box>
-      </geometry>
-    </plugin>
-    <!-- Triggers a message when the vehicle enters and exits the bay #2 -->
-    <plugin name="vehicle_docked_bay2" filename="libContainPlugin.so">
-      <entity>wamv::wamv/base_link</entity>
-      <namespace>vrx/dock_2022/bay_2</namespace>
-      <pose frame="robotx_dock_2022::dock_2022_placard2::placard::link">0 -4.5 -1.5 0 0 0</pose>
-      <geometry>
-        <box>
-          <size>1.5 4 2</size>
-        </box>
-      </geometry>
-    </plugin>
-    <plugin name="vehicle_docked_bay2_exterior" filename="libContainPlugin.so">
-      <entity>wamv::wamv/base_link</entity>
-      <namespace>vrx/dock_2022/bay_2_external</namespace>
-      <pose frame="robotx_dock_2022::dock_2022_placard2::placard::link">0 -9.5 -1.5 0 0 0</pose>
-      <geometry>
-        <box>
-          <size>5.5 1.5 2</size>
-        </box>
-      </geometry>
-    </plugin>
-    <!-- Triggers a message when the vehicle enters and exits the bay #3 -->
-    <plugin name="vehicle_docked_bay3" filename="libContainPlugin.so">
-      <entity>wamv::wamv/base_link</entity>
-      <namespace>vrx/dock_2022/bay_3</namespace>
-      <pose frame="robotx_dock_2022::dock_2022_placard3::placard::link">0 -4.5 -1.5 0 0 0</pose>
-      <geometry>
-        <box>
-          <size>1.5 4 2</size>
-        </box>
-      </geometry>
-    </plugin>
-    <plugin name="vehicle_docked_bay3_exterior" filename="libContainPlugin.so">
-      <entity>wamv::wamv/base_link</entity>
-      <namespace>vrx/dock_2022/bay_3_external</namespace>
-      <pose frame="robotx_dock_2022::dock_2022_placard3::placard::link">0 -9.5 -1.5 0 0 0</pose>
-      <geometry>
-        <box>
-          <size>5.5 1.5 2</size>
-        </box>
-      </geometry>
-    </plugin>
   </world>
 </sdf>

File: wamv_gazebo/urdf/wamv_gazebo.urdf.xacro (robot description, xacro)
@@ -138,7 +138,10 @@
       <!-- <xacro:wamv_camera name="front_left_camera" y="0.1" x="0.75" P="${radians(15)}" />
       <xacro:wamv_camera name="front_right_camera" y="-0.1" x="0.75" P="${radians(15)}" /> -->
-      <xacro:wamv_camera name="front_middle_camera" y="0.0" x="0.75" P="${radians(15)}" />
+      <!-- <xacro:wamv_camera name="front_middle_camera" y="0.0" x="0.75" P="${radians(15)}" /> -->
+      <xacro:wamv_camera name="left_camera" y="0.4" x="0.65" P="${radians(10)}" Y="${radians(30)}" post_Y="${radians(30)}"/>
+      <xacro:wamv_camera name="middle_camera" y="0" x="0.8" P="${radians(10)}" />
       <!-- Add a camera facing right -->
-      <xacro:wamv_camera name="middle_right_camera" y="-0.45" P="${radians(15)}" Y="${radians(-90)}" post_Y="${radians(-90)}" />
+      <!-- <xacro:wamv_camera name="middle_right_camera" y="-0.45" P="${radians(15)}" Y="${radians(-90)}" post_Y="${radians(-90)}" /> -->
+      <xacro:wamv_camera name="right_camera" y="-0.4" x="0.65" P="${radians(10)}" Y="${radians(-30)}" post_Y="${radians(-30)}" />
       <!-- Add simulated GPS -->
       <xacro:wamv_gps name="gps_wamv" x="-0.85" />
@@ -146,9 +149,9 @@
       <xacro:wamv_imu name="imu_wamv" y="-0.2" />
       <!-- Add 3D LIDAR -->
-      <xacro:lidar name="lidar_wamv" type="16_beam"/>
+      <xacro:lidar name="lidar_wamv" x="1.25" y="0" z="1.0" type="16_beam"/>
       <!-- Add pinger -->
-      <xacro:wamv_pinger name="pinger" position="1.0 0 -1.0" />
+      <!-- <xacro:wamv_pinger name="pinger" position="1.0 0 -1.0" /> -->
       <!-- Add ball shooter (default pitch angle: ~-60 deg) -->
-      <xacro:wamv_ball_shooter name="ball_shooter" x="0.54" y="0.30" z="1.296" pitch="-1.04"/>
+      <!-- <xacro:wamv_ball_shooter name="ball_shooter" x="0.54" y="0.30" z="1.296" pitch="-1.04"/> -->
     </xacro:if>
   </xacro:unless>

Commit message: update 05/15 on vrx

File: vrx_gazebo/worlds/master_thesis.world.xacro (robot description, xacro)
@@ -47,5 +47,5 @@
       <name>dock_2</name>
       <uri>model://dock_2022_base</uri>
-      <pose>-450 215 0 0 0 0</pose>
+      <pose>-50 215 0 0 0 0</pose>
     </include>
   </world>

File: wamv_description/urdf/wamv_base.urdf.xacro (robot description, xacro)
@@ -86,4 +86,22 @@
   <link name="${namespace}/base_link">
   </link>
+  <gazebo reference="${namespace}/base_link">
+    <sensor type="contact" name="contactsensor_sensor">
+      <always_on>true</always_on>
+      <updaterate>100.0</updaterate>
+      <contact>
+        <collision>${namespace}/base_link_fixed_joint_lump__left_float_collision_17</collision>
+        <collision>${namespace}/base_link_fixed_joint_lump__left_mid_float_collision_18</collision>
+        <collision>${namespace}/base_link_fixed_joint_lump__left_front_float_collision_19</collision>
+        <collision>${namespace}/base_link_fixed_joint_lump__right_float_collision_29</collision>
+        <collision>${namespace}/base_link_fixed_joint_lump__right_mid_float_collision_30</collision>
+        <collision>${namespace}/base_link_fixed_joint_lump__right_front_float_collision_31</collision>
+      </contact>
+      <plugin name="gazebo_ros_bumper_controller" filename="libgazebo_ros_bumper.so">
+        <bumperTopicName>${namespace}/bumper_states</bumperTopicName>
+        <frameName>world</frameName>
+      </plugin>
+    </sensor>
+  </gazebo>
   <joint name="${namespace}/dummy_joint" type = "fixed">
     <parent link="${namespace}/base_link"/>

Commit message: on vrx

File: vrx_gazebo/worlds/master_thesis.world.xacro (robot description, xacro)
@@ -49,4 +49,9 @@
       <pose>-50 215 0 0 0 0</pose>
     </include>
+    <include>
+      <name>obstacle_1</name>
+      <uri>model://obstacle_course1</uri>
+      <pose>-525 219 0.11 0 0 0</pose>
+    </include>
   </world>
 </sdf>

File: wave_gazebo/world_models/ocean_waves/model.xacro (robot description, xacro)
@@ -17,5 +17,5 @@
 -->
 <world xmlns:xacro="http://ros.org/wiki/xacro">
-  <xacro:macro name="ocean_waves" params="gain:=0.7 period:=5
+  <xacro:macro name="ocean_waves" params="gain:=0.1 period:=5
                      direction_x:=1.0 direction_y:=0.0
                      angle:=0.4 scale:=1.5">
